File: table_nixeClock_IN-8_PCB/shemLamps.brd (EAGLE design)
At the start: 170 x 50 mm, 84 parts, among them IC1 K155ID1, IC2 74HC595, IC4 STM8S003F3, J1 DCJ0202, Q2 SPD06N80C3, T1 PMBTA42, T10 MMBTA92, T11 PMBTA42, T12 MMBTA92, T13 PMBTA42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

Commit message: RealeaseV2.2
Parts:
- added C7, C8: 12pf, myRlc:C0805
- added C9: 100nf, myRlc:C0805
- C4: value 100nf -> 10nf
- C6: value 10uf/400V -> 2.2uf/400V
- IC4: value STM8S003F3 -> STM8S003; device inter:TSSOP20 -> inter:TSSOP-20
- L1: value 240u -> 270u
- Q1: value (none) -> 32.768kHz
- R1, R2: value 51k -> 100k
Connections:
- net GND: now also C7.1, C8.1, C9.1
- net N$32: now also C8.2
- net N$36: now also C7.2
- net VCC: now also C9.2
Routing:
- net N$32: track 8.30 -> 11.5 mm
- net N$36: track 2.32 -> 4.71 mm
- net VCC: track 234.2 -> 234.7 mm
- net PWM: track 68.4 -> 68.9 mm
- net OK: track 51.1 -> 51.6 mm
- net NRS_MCU: track 25.4 -> 25.9 mm
- net I2C_CLK: track 18.4 -> 18.9 mm
- net DOWN: track 63.1 -> 63.6 mm
- net D3: track 69.6 -> 70.1 mm
- net D2: track 56.6 -> 57.1 mm
- net D1: track 65.3 -> 65.8 mm
- net D0: track 71.2 -> 71.7 mm
Other:
- board text removed: "01-16"
- board text removed: "01-20"
- board text removed: "LAYER-STACK"
