File: table_nixeClock_IN-8_PCB/shemLamps.sch (EAGLE design)
At the start: 84 parts, among them IC1 K155ID1, IC2 74HC595, IC4 STM8S003F3, J1 DCJ0202, Q2 SPD06N80C3, T1 PMBTA42, T10 MMBTA92, T11 PMBTA42, T12 MMBTA92, T13 PMBTA42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

Commit message: RealeaseV2.2
Parts:
- added C7, C8: 12pf, myRlc:CAP
- added C9: 100nf, myRlc:CAP
- C4: value 100nf -> 10nf
- C6: value 10uf/400V -> 2.2uf/400V
- IC4: value STM8S003F3 -> STM8S003; device inter:STM8S003F3 -> inter:STM8S003
- L1: value 240u -> 270u
- Q1: value (none) -> 32.768kHz
- R1, R2: value 51k -> 100k
Connections:
- net GND: now also C7.1, C8.1, C9.1
- net N$32: now also C8.2
- net N$36: now also C7.2
- net VCC: now also C9.2, IC4.VCC; no longer IC4.VDD
Changed lines of the file:
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@@
 <part name="SUPPLY1" library="supply2" library_urn="urn:adsk.eagle:library:372" deviceset="GND" device=""/>
 <part name="SUPPLY2" library="supply2" library_urn="urn:adsk.eagle:library:372" deviceset="GND" device=""/>
-<part name="R1" library="rcl" library_urn="urn:adsk.eagle:library:334" deviceset="R-EU_" device="0207/10" package3d_urn="urn:adsk.eagle:package:23491/2" value="51k"/>
-<part name="R2" library="rcl" library_urn="urn:adsk.eagle:library:334" deviceset="R-EU_" device="0207/10" package3d_urn="urn:adsk.eagle:package:23491/2" value="51k"/>
+<part name="R1" library="rcl" library_urn="urn:adsk.eagle:library:334" deviceset="R-EU_" device="0207/10" package3d_urn="urn:adsk.eagle:package:23491/2" value="100k"/>
+<part name="R2" library="rcl" library_urn="urn:adsk.eagle:library:334" deviceset="R-EU_" device="0207/10" package3d_urn="urn:adsk.eagle:package:23491/2" value="100k"/>
 <part name="J1" library="con-jack" library_urn="urn:adsk.eagle:library:154" deviceset="DCJ0202" device="" package3d_urn="urn:adsk.eagle:package:7491/1"/>
 <part name="SUPPLY3" library="supply2" library_urn="urn:adsk.eagle:library:372" deviceset="GND" device=""/>
@@
 <part name="P+3" library="supply1" library_urn="urn:adsk.eagle:library:371" deviceset="VCC" device=""/>
 <part name="C2" library="myRlc" deviceset="CAP" device="" package3d_urn="urn:adsk.eagle:package:23617/2" value="100nf"/>
-<part name="IC4" library="inter" deviceset="STM8S003" device="F3"/>
+<part name="IC4" library="inter" deviceset="STM8S003" device="" value="STM8S003"/>
 <part name="SUPPLY17" library="supply2" library_urn="urn:adsk.eagle:library:372" deviceset="GND" device=""/>
 <part name="P+6" library="supply1" library_urn="urn:adsk.eagle:library:371" deviceset="VCC" device=""/>
@@
 <part name="P+7" library="supply1" library_urn="urn:adsk.eagle:library:371" deviceset="VCC" device=""/>
 <part name="SUPPLY18" library="supply2" library_urn="urn:adsk.eagle:library:372" deviceset="GND" device=""/>
-<part name="C4" library="myRlc" deviceset="CAP" device="" package3d_urn="urn:adsk.eagle:package:23617/2" value="100nf"/>
+<part name="C4" library="myRlc" deviceset="CAP" device="" package3d_urn="urn:adsk.eagle:package:23617/2" value="10nf"/>
 <part name="R40" library="myRlc" deviceset="RES" device="" package3d_urn="urn:adsk.eagle:package:23553/2" value="1k"/>
 <part name="P+8" library="supply1" library_urn="urn:adsk.eagle:library:371" deviceset="VCC" device=""/>
@@
 <part name="U1" library="inter" deviceset="DS1307" device="" package3d_urn="urn:adsk.eagle:package:39057/1"/>
 <part name="SUPPLY20" library="supply2" library_urn="urn:adsk.eagle:library:372" deviceset="GND" device=""/>
-<part name="Q1" library="crystal" library_urn="urn:adsk.eagle:library:204" deviceset="CRYSTAL" device="TC26H" package3d_urn="urn:adsk.eagle:package:12086/1"/>
+<part name="Q1" library="crystal" library_urn="urn:adsk.eagle:library:204" deviceset="CRYSTAL" device="TC26H" package3d_urn="urn:adsk.eagle:package:12086/1" value="32.768kHz"/>
 <part name="P+9" library="supply1" library_urn="urn:adsk.eagle:library:371" deviceset="VCC" device=""/>
 <part name="C5" library="myRlc" deviceset="CAP" device="" package3d_urn="urn:adsk.eagle:package:23617/2" value="100nf"/>
@@
 <part name="SUPPLY15" library="supply2" library_urn="urn:adsk.eagle:library:372" deviceset="GND" device=""/>
 <part name="D1" library="diode" library_urn="urn:adsk.eagle:library:210" deviceset="DIODE-" device="DO-214AC" package3d_urn="urn:adsk.eagle:package:43416/2" value="GS1M"/>
-<part name="L1" library="inductor-neosid" library_urn="urn:adsk.eagle:library:241" deviceset="BS" device="11" package3d_urn="urn:adsk.eagle:package:14648/1" value="240u"/>
+<part name="L1" library="inductor-neosid" library_urn="urn:adsk.eagle:library:241" deviceset="BS" device="11" package3d_urn="urn:adsk.eagle:package:14648/1" value="270u"/>
 <part name="P+4" library="supply1" library_urn="urn:adsk.eagle:library:371" deviceset="VCC" device=""/>
-<part name="C6" library="rcl" library_urn="urn:adsk.eagle:library:334" deviceset="CPOL-EU" device="E3.5-8" package3d_urn="urn:adsk.eagle:package:23360/2" value="10uf/400V"/>
+<part name="C6" library="rcl" library_urn="urn:adsk.eagle:library:334" deviceset="CPOL-EU" device="E3.5-8" package3d_urn="urn:adsk.eagle:package:23360/2" value="2.2uf/400V"/>
 <part name="SUPPLY16" library="supply2" library_urn="urn:adsk.eagle:library:372" deviceset="GND" device=""/>
 <part name="Q2" library="inter" deviceset="SPD06N80C3" device="" package3d_urn="urn:adsk.eagle:package:28537/2"/>
 <part name="R39" library="myRlc" deviceset="RES" device="" package3d_urn="urn:adsk.eagle:package:23553/2" value="10k"/>
 <part name="R41" library="myRlc" deviceset="RES" device="" package3d_urn="urn:adsk.eagle:package:23553/2" value="10k"/>
+<part name="C7" library="myRlc" deviceset="CAP" device="" package3d_urn="urn:adsk.eagle:package:23617/2" value="12pf"/>
+<part name="C8" library="myRlc" deviceset="CAP" device="" package3d_urn="urn:adsk.eagle:package:23617/2" value="12pf"/>
+<part name="SUPPLY22" library="supply2" library_urn="urn:adsk.eagle:library:372" deviceset="GND" device=""/>
+<part name="C9" library="myRlc" deviceset="CAP" device="" package3d_urn="urn:adsk.eagle:package:23617/2" value="100nf"/>
 </parts>
 <sheets>
@@
 </instance>
 <instance part="Q1" gate="G$1" x="228.6" y="50.8" smashed="yes" rot="MR270">
-<attribute name="NAME" x="227.584" y="48.26" size="1.778" layer="95" rot="MR270"/>
-<attribute name="VALUE" x="231.14" y="48.26" size="1.778" layer="96" rot="MR270"/>
+<attribute name="NAME" x="226.314" y="54.61" size="1.778" layer="95" rot="MR90"/>
+<attribute name="VALUE" x="229.87" y="54.61" size="1.778" layer="96" rot="MR90"/>
 </instance>
 <instance part="P+9" gate="VCC" x="261.62" y="60.96" smashed="yes">
@@
 <attribute name="NAME" x="272.8214" y="46.99" size="1.778" layer="95" rot="R90"/>
 <attribute name="VALUE" x="277.622" y="46.99" size="1.778" layer="96" rot="R90"/>
+</instance>
+<instance part="C7" gate="G$1" x="218.44" y="53.34" smashed="yes" rot="R90">
+<attribute name="NAME" x="218.059" y="54.864" size="1.778" layer="95" rot="R90"/>
+<attribute name="VALUE" x="223.139" y="54.864" size="1.778" layer="96" rot="R90"/>
+</instance>
+<instance part="C8" gate="G$1" x="218.44" y="45.72" smashed="yes" rot="R90">
+<attribute name="NAME" x="218.059" y="47.244" size="1.778" layer="95" rot="R90"/>
+<attribute name="VALUE" x="223.139" y="47.244" size="1.778" layer="96" rot="R90"/>
+</instance>
+<instance part="SUPPLY22" gate="GND" x="213.36" y="40.64" smashed="yes">
+<attribute name="VALUE" x="211.455" y="37.465" size="1.778" layer="96"/>
+</instance>
+<instance part="C9" gate="G$1" x="17.78" y="45.72" smashed="yes" rot="R180">
+<attribute name="NAME" x="16.256" y="45.339" size="1.778" layer="95" rot="R180"/>
+<attribute name="VALUE" x="16.256" y="50.419" size="1.778" layer="96" rot="R180"/>
 </instance>
 </instances>
@@
 <pinref part="C4" gate="G$1" pin="2"/>
 <junction x="27.94" y="38.1"/>
+<pinref part="C9" gate="G$1" pin="1"/>
+<wire x1="17.78" y1="43.18" x2="17.78" y2="38.1" width="0.1524" layer="91"/>
+<wire x1="17.78" y1="38.1" x2="27.94" y2="38.1" width="0.1524" layer="91"/>
 </segment>
 <segment>
@@
 <pinref part="C6" gate="G$1" pin="-"/>
 <wire x1="132.08" y1="96.52" x2="132.08" y2="99.06" width="0.1524" layer="91"/>
+</segment>
+<segment>
+<pinref part="C8" gate="G$1" pin="1"/>
+<wire x1="215.9" y1="45.72" x2="213.36" y2="45.72" width="0.1524" layer="91"/>
+<pinref part="C7" gate="G$1" pin="1"/>
+<wire x1="213.36" y1="45.72" x2="213.36" y2="53.34" width="0.1524" layer="91"/>
+<wire x1="213.36" y1="53.34" x2="215.9" y2="53.34" width="0.1524" layer="91"/>
+<pinref part="SUPPLY22" gate="GND" pin="GND"/>
+<wire x1="213.36" y1="43.18" x2="213.36" y2="45.72" width="0.1524" layer="91"/>
+<junction x="213.36" y="45.72"/>
 </segment>
 </net>
@@
 <segment>
 <pinref part="P+6" gate="VCC" pin="VCC"/>
-<pinref part="IC4" gate="G$1" pin="VDD"/>
+<pinref part="IC4" gate="G$1" pin="VCC"/>
 <wire x1="27.94" y1="73.66" x2="27.94" y2="68.58" width="0.1524" layer="91"/>
 <wire x1="27.94" y1="68.58" x2="27.94" y2="50.8" width="0.1524" layer="91"/>
@@
 <wire x1="30.48" y1="68.58" x2="27.94" y2="68.58" width="0.1524" layer="91"/>
 <junction x="27.94" y="68.58"/>
+<pinref part="C9" gate="G$1" pin="2"/>
+<wire x1="17.78" y1="50.8" x2="27.94" y2="50.8" width="0.1524" layer="91"/>
+<junction x="27.94" y="50.8"/>
 </segment>
 <segment>
@@
 <pinref part="Q1" gate="G$1" pin="2"/>
 <wire x1="228.6" y1="48.26" x2="228.6" y2="45.72" width="0.1524" layer="91"/>
+<pinref part="C8" gate="G$1" pin="2"/>
+<wire x1="223.52" y1="45.72" x2="228.6" y2="45.72" width="0.1524" layer="91"/>
+<junction x="228.6" y="45.72"/>
 </segment>
 </net>
@@
 <pinref part="Q1" gate="G$1" pin="1"/>
 <wire x1="228.6" y1="53.34" x2="233.68" y2="53.34" width="0.1524" layer="91"/>
-</segment>
-</net>
+<pinref part="C7" gate="G$1" pin="2"/>
+<wire x1="223.52" y1="53.34" x2="228.6" y2="53.34" width="0.1524" layer="91"/>
+<junction x="228.6" y="53.34"/>
+</segment>
+</net>
